File: Hardware/MeshLoRa/_autosave-SX1262.kicad_sch (KiCad schematic)
At the start: 1 part

Commit message: Added SX1262 Schematic + Footprint
Added SX1262 Schematic + Footprint
Parts:
- U?: footprint QFN50P400X400X100-25N -> SX1262:QFN50P400X400X100-25N
Changed lines of the file:
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@@
     (property "Reference" "U?" (id 0) (at 135.382 50.3895 0))
     (property "Value" "SX1262IMLTRT" (id 1) (at 135.382 53.1646 0))
-    (property "Footprint" "QFN50P400X400X100-25N" (id 2) (at 135.382 82.296 0)
+    (property "Footprint" "SX1262:QFN50P400X400X100-25N" (id 2) (at 135.382 82.296 0)
       (effects (font (size 1.27 1.27)) (justify bottom) hide)
     )
