File: Hardware/boards/Mesh_v1/Mesh_v1.kicad_sch (KiCad schematic)
At the start: 54 parts

Commit message: Nearly finished sch
Parts:
- removed BT?: 18650, Battery:BatteryHolder_Keystone_1042_1x18650, symbol Device:Battery_Cell
- removed D?: PTZTFTE255.1B, Diode_SMD:D_SMF, symbol Device:D_Zener
- removed J?: Conn_01x03, Connector_PinHeader_2.54mm:PinHeader_1x03_P2.54mm_Vertical, symbol Connector_Generic:Conn_01x03
- removed J?: Molex Micro-Lock 5055780271, Connector_Molex:Molex_CLIK-Mate_502494-0270_1x02-1MP_P2.00mm_Horizontal, symbol Connector_Generic:Conn_01x02
- removed J?: Conn_01x05, Connector_PinHeader_2.54mm:PinHeader_1x01_P2.54mm_Vertical, symbol Connector_Generic:Conn_01x01
- removed J? (x2): Conn_01x02, Connector_PinHeader_2.54mm:PinHeader_1x02_P2.54mm_Vertical, symbol Connector_Generic:Conn_01x02
- removed J?: Molex Micro-Fit 436500200, Connector_Molex:Molex_Micro-Fit_3.0_43650-0200_1x02_P3.00mm_Horizontal, symbol Connector_Generic:Conn_01x02
- removed R?: 30k, Resistor_SMD:R_0805_2012Metric, symbol Device:R_US
- removed U?: USBLC6-2P6, Package_TO_SOT_SMD:SOT-666, symbol Power_Protection:USBLC6-2P6
- added C108: 1uF, symbol Device:C
- added C109: 10uF, symbol Device:C
- added D101: MBR120, Diode_SMD:D_SOD-123F, symbol Device:D_Schottky
- added J103, J106: Conn_01x03, Connector_PinHeader_2.54mm:PinHeader_1x03_P2.54mm_Vertical, symbol Connector_Generic:Conn_01x03
- added J104: Conn_01x02, Connector_PinHeader_2.54mm:PinHeader_1x02_P2.54mm_Vertical, symbol Connector_Generic:Conn_01x02
- added J105: Conn_01x05, Connector_PinHeader_2.54mm:PinHeader_1x01_P2.54mm_Vertical, symbol Connector_Generic:Conn_01x01
- added J109: USB_B_Micro, Connector_USB:USB_Micro-B_Molex_47346-0001, symbol Connector:USB_B_Micro
- added R106: 22.1K, symbol Device:R_US
- added R107: 47.5K, symbol Device:R_US
- added R110: 1K, symbol Device:R_US
- added U105: CP2102N-Axx-xQFN28, Package_DFN_QFN:QFN-28-1EP_5x5mm_P0.5mm_EP3.35x3.35mm, symbol Interface_USB:CP2102N-Axx-xQFN28
- D102: renamed from D?; value Orange -> Red
- J102: renamed from J?; footprint Connector_Molex:Molex_Micro-Fit_3.0_43650-0200_1x02_P3.00mm_Horizontal -> Connector_JST:JST_PH_B2B-PH-K_1x02_P2.00mm_Vertical
- gave numbers to parts that had none: 42
Connections:
- net +BATT is gone; now on net VBAT: C107.1, U104.3 (VBAT)
- net 5V is gone; now on net VBUS: J108.1 (VBUS)
- net PSU_RAW is gone; now on net VBAT: J102.1 (Pin_1)
- net 3V3: now also C109.1, J106.1 (Pin_1), R110.2, U105.6 (VDD), U105.7 (VREGIN)
- net ESP_USB_DN: now also J108.2 (D-)
- net ESP_USB_DP: now also J108.3 (D+)
- net GND: now also C108.2, C109.2, J106.2 (Pin_2), J109.5 (GND), J109.6 (Shield), R107.1, U105.29 (GND), U105.3 (GND)
- net LED_BLUE: now also U106.33 (IO40); no longer U106.34 (IO41)
- net LED_GREEN: now also U106.34 (IO41); no longer U106.35 (IO42)
- net LED_ORANGE: now also U106.35 (IO42); no longer U106.36 (RXD0)
- net LED_RED: no longer U106.37 (TXD0)
- net RADIO_SPI_MISO: now also J103.1 (Pin_1)
- net RADIO_SPI_MOSI: now also J103.2 (Pin_2)
- net RADIO_SPI_SCK: now also J103.3 (Pin_3)
- net RFM96W_CS: now also J105.1 (Pin_1)
- net TELEM_I2C_SCL: now also J104.1 (Pin_1)
- net TELEM_I2C_SDA: now also J104.2 (Pin_2)
- net VBAT: now also D101.2 (A), J106.3 (Pin_3); no longer C102.1, C105.1, C106.1, U103.1 (VIN)
- net VBUS: now reaches D102.2 (A), U104.4 (VDD)
- net VBUS: now also C102.1, C105.1, C106.1, U103.1 (VIN), D101.1 (K)
- new net: R106.1, U105.8 (VBUS)
- new net: R110.1, U105.24 (~{RTS})
- new net RX_UART_USB: U105.25 (RXD), U106.37 (TXD0)
- new net TX_UART_USB: U105.26 (TXD), U106.36 (RXD0)
- new net UART_USB_DN: J109.2 (D-), U105.5 (D-)
- new net UART_USB_DP: J109.3 (D+), U105.4 (D+)
- new net VBUS_UART: C108.1, J109.1 (VBUS), R106.2, R107.2
- no-connect marks 14 -> 22
Other:
- note added: "18650 Battery"
- note added: "1S1P 18650 3.7V"
- note added: "Battery Voltage Range Single: 3V-4.2V"
- note added: "ESP32 USB/UART Port"
- note added: "PROG Charging Rate 10K = 100mA 5K = 200mA 2K = 500mA 1K = 1000mA"
- note added: "Power"
- note added: "USB Lipo Charger"
- note removed: "!!!WARNING: DISCONNECT BATTERIES BEFORE USE!!!"
- note removed: "18650 3.7V Batteries x6"
- note removed: "2S1P 7.4V Battery Pack"
- note removed: "2S2P 7.4V Battery Pack"
- note removed: "2S3P 18650 7.4V"
- note removed: "7.4V Typical, 8.4V MAX, 35W MAX"
- note removed: "Battery Voltage Range Single: 3V-4.2V Total: 6V-8.4V"
- note removed: "Bench Power Supply"
- note removed: "Included ESD Protection"
- note removed: "Screw Switch"
- title: (none) -> Mesh Board MK1
- moved on the sheet: C101, C102, C104, C105, C106, C107, C110, C111, C112, C113, C114, D102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
