File: Hardware/Breakouts/ESP32/ESP32.kicad_sch (KiCad schematic)
At the start: 2 parts

Commit message: stuff part 3
Parts:
- added U?: W25Q128JVS, Package_SO:SOIC-8_5.23x5.23mm_P1.27mm, symbol Memory_Flash:W25Q128JVS
- U?: MPN (none) -> ESP32-D0WD-V3
Changed lines of the file:
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@@
+      (effects (font (size 1.27 1.27)) hide)
+    )
+    (property "MPN" "ESP32-D0WD-V3" (id 4) (at 147.32 101.6 0)
       (effects (font (size 1.27 1.27)) hide)
     )
@@
     (pin "9")
   )
+  (symbol (lib_id "Memory_Flash:W25Q128JVS") (at 59.69 83.82 0) (unit 1)
+    (in_bom yes) (on_board yes) (fields_autoplaced)
+    (property "Reference" "U?" (id 0) (at 61.7094 71.12 0)
+      (effects (font (size 1.27 1.27)) (justify left))
+    )
+    (property "Value" "W25Q128JVS" (id 1) (at 61.7094 73.66 0)
+      (effects (font (size 1.27 1.27)) (justify left))
+    )
+    (property "Footprint" "Package_SO:SOIC-8_5.23x5.23mm_P1.27mm" (id 2) (at 59.69 83.82 0)
+      (effects (font (size 1.27 1.27)) hide)
+    )
+    (property "Datasheet" "http://www.winbond.com/resource-files/w25q128jv_dtr%20revc%2003272018%20plus.pdf" (id 3) (at 59.69 83.82 0)
+      (effects (font (size 1.27 1.27)) hide)
+    )
+    (property "MPN" "W25Q128JVSIQ" (id 4) (at 59.69 83.82 0)
+      (effects (font (size 1.27 1.27)) hide)
+    )
+    (pin "1")
+    (pin "2")
+    (pin "3")
+    (pin "4")
+    (pin "5")
+    (pin "6")
+    (pin "7")
+    (pin "8")
+  )
   (symbol (lib_id "Regulator_Linear:LM1117-3.3") (at 72.39 130.81 0) (unit 1)
     (in_bom yes) (on_board yes) (fields_autoplaced)
@@
       (reference "U?") (unit 1) (value "ESP32") (footprint "Package_DFN_QFN:QFN-48-1EP_5x5mm_P0.35mm_EP3.7x3.7mm")
     )
+    (path "/3705ffba-1848-4055-9880-0fe6a15e73ca"
+      (reference "U?") (unit 1) (value "W25Q128JVS") (footprint "Package_SO:SOIC-8_5.23x5.23mm_P1.27mm")
+    )
     (path "/8ccd251c-dc8c-4375-b705-06f42ceab9a8"

Commit message: did schematic almost done
Parts:
- added AE1: Antenna, symbol Device:Antenna
- added C1, C2, C4, C6, C7, C8, C? (x2): 100n, Capacitor_SMD:C_0805_2012Metric, symbol Device:C
- added C3, C5: C, symbol Device:C
- added C?: C, Capacitor_SMD:C_0805_2012Metric, symbol Device:C
- added C?: 8p, Capacitor_SMD:C_0805_2012Metric, symbol Device:C
- added C?: 10n, Capacitor_SMD:C_0805_2012Metric, symbol Device:C
- added C? (x2): 10u, Capacitor_SMD:C_1206_3216Metric, symbol Device:C
- added C?: 3.3n, Capacitor_SMD:C_0805_2012Metric, symbol Device:C
- added C?: 1u, Capacitor_SMD:C_0805_2012Metric, symbol Device:C
- added FB?: FerriteBead, Resistor_SMD:R_0805_2012Metric, symbol Device:FerriteBead
- added J?: USB_B_Micro, Connector_USB:USB_Micro-B_GCT_USB3076-30-A, symbol Connector:USB_B_Micro
- added JP?: Jumper_2_Open, Jumper:SolderJumper-2_P1.3mm_Open_RoundedPad1.0x1.5mm, symbol Jumper:Jumper_2_Open
- added L1: L, symbol Device:L
- added R1: 0, Resistor_SMD:R_0805_2012Metric, symbol Device:R_US
- added R?: 1k, Resistor_SMD:R_0805_2012Metric, symbol Device:R_US
- added R?: 20k, Resistor_SMD:R_0805_2012Metric, symbol Device:R_US
- added U?: CP2104, Package_DFN_QFN:QFN-24-1EP_4x4mm_P0.5mm_EP2.6x2.6mm, symbol Interface_USB:CP2104
- added Y?: Crystal_GND24, Crystal:Crystal_SMD_2016-4Pin_2.0x1.6mm, symbol Device:Crystal_GND24
- gave numbers to parts that had none: 3
Connections:
- net at U2.1 (VDDA), U2.43 (VDDA), U2.46 (VDDA): now also C?.1, C?.1, FB?.2
- net +3V3: now reaches U2.19 (VDD3P3_RTC)
- net +3V3: now also U1.2 (VO), U2.3 (VDD3P3), U2.37 (VDD3P3_CPU), U2.4 (VDD3P3), C1.1, C2.1, C4.1, C6.1, C7.1, C?.1, FB?.1, JP?.2 (B)
- net at U2.2 (LNA_IN): now also C5.1, L1.2
- net IO2: now reaches U2.22 (GPIO2/ADC2_CH2)
- net IO0: now reaches U2.23 (GPIO0/BOOT/ADC2_CH1)
- net IO4: now reaches U2.24 (GPIO4/ADC2_CH0)
- net VDD_SDIO: now reaches U2.26 (VDD_SDIO)
- net VDD_SDIO: now also U3.8 (VCC), C8.1, C?.1, JP?.1 (A)
- net FLASH_IO2: now reaches U2.28 (SD_DATA_2/GPIO9)
- net FLASH_IO2: now also U3.3 (IO2)
- net FLASH_IO3: now reaches U2.29 (SD_DATA_3/GPIO10)
- net FLASH_IO3: now also U3.7 (IO3)
- net FLASH_CS: now reaches U2.30 (SD_CMD/GPIO11)
- net FLASH_CS: now also U3.1 (~{CS})
- net FLASH_CLK: now reaches U2.31 (SD_CLK/GPIO6)
- net FLASH_CLK: now also U3.6 (CLK)
- net FLASH_IO1: now reaches U2.32 (SD_DATA_0/GPIO7)
- net FLASH_IO1: now also U3.2 (DO(IO1))
- net FLASH_IO0: now reaches U2.33 (SD_DATA_1/GPIO8)
- net FLASH_IO0: now also U3.5 (DI(IO0))
- net IO5: now reaches U2.34 (GPIO5)
- net RXD: now reaches U2.40 (U0RXD/GPIO3)
- net RXD: now also U?.20 (RXD)
- net TXD: now reaches U2.41 (U0TXD/GPIO1)
- net TXD: now also U?.21 (TXD)
- net at U2.44 (XTAL_N): now also C?.2, Y?.3
- net at U2.45 (XTAL_P): now also R?.2
- net at U2.47 (CAP2): now also C?.2, R?.2
- net at U2.48 (CAP1): now also C?.1, C?.1, R?.1
- net GND: now reaches U2.49 (GND)
- net GND: now also U1.1 (GND), U3.4 (GND), C1.2, C2.2, C3.2, C4.2, C5.2, C6.2, C7.2, C8.2, C?.1, C?.1, C?.2, C?.2, C?.2, C?.2, C?.2, C?.2, J?.5 (GND), J?.6 (Shield), U?.2 (GND), U?.25 (GND), Y?.2, Y?.4
- net EN: now reaches U2.9 (CHIP_PU)
- net EN: now also C?.1
- net VBUS: now reaches U1.3 (VI)
- net VBUS: now also J?.1 (VBUS), U?.7 (REGIN)
- new net: C3.1, L1.1, R1.2
- new net: AE1.1 (A), R1.1
- new net: C?.2, R?.1, Y?.1
- new net: J?.2 (D-), U?.4 (D-)
- new net: J?.3 (D+), U?.3 (D+)
- new net +5V: U?.8 (VBUS)
- new net DSR: U?.22 (~{DSR})
- new net DTR: U?.23 (~{DTR})
Other:
- moved on the sheet: U1, U2, U3

Commit message: satuff
Parts:
- removed C?: 10n, Capacitor_SMD:C_0805_2012Metric, symbol Device:C
- removed C?: 3.3n, Capacitor_SMD:C_0805_2012Metric, symbol Device:C
- removed R?: 20k, Resistor_SMD:R_0805_2012Metric, symbol Device:R_US
- removed U1: LM1117-3.3, symbol Regulator_Linear:LM1117-3.3
- removed U?: CP2104, Package_DFN_QFN:QFN-24-1EP_4x4mm_P0.5mm_EP2.6x2.6mm, symbol Interface_USB:CP2104
- added J1: Conn_02x20_Odd_Even, Connector_PinHeader_2.54mm:PinHeader_2x20_P2.54mm_Vertical, symbol Connector_Generic:Conn_02x20_Odd_Even
- added Q1, Q2: BC817, Package_TO_SOT_SMD:SOT-23, symbol Transistor_BJT:BC817
- added R4, R5, R6, R7, R8, R9: 10k, Resistor_SMD:R_0805_2012Metric, symbol Device:R_US
- added U1: AMS1117-3.3, Package_TO_SOT_SMD:SOT-223-3_TabPin2, symbol Regulator_Linear:AMS1117-3.3
- added U4: CP2102N-Axx-xQFN24, Package_DFN_QFN:QFN-24-1EP_4x4mm_P0.5mm_EP2.6x2.6mm, symbol Interface_USB:CP2102N-Axx-xQFN24
- AE1: footprint (none) -> Connector_Coaxial:U.FL_Hirose_U.FL-R-SMT-1_Vertical; MPN (none) -> U.FL-R-SMT-1(80)
- C1, C2, C4, C6, C7, C8: MPN (none) -> CL21B104KBCNNNC
- C10: renamed from C?; value C -> 8p; MPN (none) -> 08051A8R0DAT2A
- C13, C17: renamed from C?; MPN (none) -> CL21B104KBCNNNC
- C14: renamed from C?; MPN (none) -> CL21B105KAFNNNE
- C15, C16: renamed from C?; MPN (none) -> CL31A106KQHNNNE
- C3, C5: footprint (none) -> Capacitor_SMD:C_0603_1608Metric; MPN (none) -> CBR06C609B5GAC
- C9: renamed from C?; MPN (none) -> 08051A8R0DAT2A
- FB1: renamed from FB?; MPN (none) -> 2508056017Y2
- L1: value L -> 0.6n; footprint (none) -> Inductor_SMD:L_0603_1608Metric; MPN (none) -> LQP03HQ0N6W02D
- R1: value 0 -> 22.1k; MPN (none) -> RC0805FR-0722K1L
- R3: renamed from R?; MPN (none) -> RNCP0805FTD1K00
- gave numbers to parts that had none: 3
Connections:
- net +3V3: now also J1.1 (Pin_1), J1.2 (Pin_2), R4.2, U1.2 (VO), U4.5 (VIO), U4.6 (VDD), U4.9 (~{RST})
- net DSR: now also U4.22 (~{DSR})
- net DTR: now also Q2.2 (E), R5.1, U4.23 (~{DTR})
- net EN: now also Q1.3 (C)
- net FLASH_CS: now also R4.1
- net GND: now also J1.39 (Pin_39), J1.40 (Pin_40), R7.1, U1.1 (GND), U4.2 (GND), U4.25 (GND)
- net IO0: now also Q2.3 (C)
- net IO2: now also J1.3 (Pin_3), J1.4 (Pin_4)
- net IO4: now also J1.5 (Pin_5), J1.6 (Pin_6)
- net IO5: now also J1.7 (Pin_7), J1.8 (Pin_8)
- net RXD: now also R9.2
- net TXD: now also R8.2
- net VBUS: now also R1.2, U1.3 (VI)
- net IO34: now reaches U2.10 (VDET_1/GPIO34/ADC1_CH6)
- net IO35: now reaches U2.11 (VDET_2/GPIO35/ADC1_CH7)
- net IO32: now reaches U2.12 (32K_XP/GPIO32/ADC1_CH4)
- net IO33: now reaches U2.13 (32K_XN/GPIO33/ADC1_CH5)
- net IO25: now reaches U2.14 (GPIO25/ADC2_CH8/DAC_1)
- net IO25: now also J1.19 (Pin_19), J1.20 (Pin_20)
- net IO26: now reaches U2.15 (GPIO26/ADC2_CH9/DAC_2)
- net IO26: now also J1.21 (Pin_21), J1.22 (Pin_22)
- net IO27: now reaches U2.16 (GPIO27/ADC2_CH7)
- net IO27: now also J1.23 (Pin_23), J1.24 (Pin_24)
- net IO14: now reaches U2.17 (MTMS/GPIO14/ADC2_CH6)
- net IO14: now also J1.25 (Pin_25), J1.26 (Pin_26)
- net IO12: now reaches U2.18 (MTDI/GPIO12/ADC2_CH5)
- net IO12: now also J1.27 (Pin_27), J1.28 (Pin_28)
- net IO13: now reaches U2.20 (MTCK/GPIO13/ADC2_CH4)
- net IO13: now also J1.29 (Pin_29), J1.30 (Pin_30)
- net IO15: now reaches U2.21 (MTDO/GPIO15/ADC2_CH3)
- net IO15: now also J1.31 (Pin_31), J1.32 (Pin_32)
- net IO16: now reaches U2.25 (GPIO16)
- net IO17: now reaches U2.27 (GPIO17)
- net IO18: now reaches U2.35 (GPIO18)
- net IO18: now also J1.10 (Pin_10), J1.9 (Pin_9)
- net IO23: now reaches U2.36 (GPIO23)
- net IO23: now also J1.17 (Pin_17), J1.18 (Pin_18)
- net IO19: now reaches U2.38 (GPIO19)
- net IO19: now also J1.11 (Pin_11), J1.12 (Pin_12)
- net IO22: now reaches U2.39 (GPIO22)
- net IO22: now also J1.15 (Pin_15), J1.16 (Pin_16)
- net IO21: now reaches U2.42 (GPIO21)
- net IO21: now also J1.13 (Pin_13), J1.14 (Pin_14)
- net IO36: now reaches U2.5 (SENSOR_VP/GPIO36/ADC1_CH0)
- net IO37: now reaches U2.6 (SENSOR_CAPP/GPIO37/ADC1_CH1)
- net IO38: now reaches U2.7 (SENSOR_CAPN/GPIO38/ADC1_CH2)
- net IO39: now reaches U2.8 (SENSOR_VN/GPIO39/ADC1_CH3)
- net at C3.1, L1.1: now also AE1.1 (A); no longer R1.2
- net at R1.1: now also R7.2, U4.8 (VBUS); no longer AE1.1 (A)
- net at J2.2 (D-): now also U4.4 (D-)
- net at J2.3 (D+): now also U4.3 (D+)
- new net: Q1.1 (B), R5.2
- new net: R9.1, U4.20 (RXD)
- new net: Q2.1 (B), R6.2
- new net: R8.1, U4.21 (TXD)
- new net RTS: Q1.2 (E), R6.1, U4.19 (~{RTS})
Other:
- moved on the sheet: C14, C17, C8, JP1, U3
